Commit message: Added all needed for the video response

File: plannar_mover/urdf/plannar_mover.urdf (robot description, URDF)
Before this commit: robot gurdy, 11 links, 10 joints
Links:
- removed link base_link
- removed link footM1_link
- removed link footM2_link
- removed link footM3_link
- removed link head_link
- removed link lowerleg_M1_link
- removed link lowerleg_M2_link
- removed link lowerleg_M3_link
- removed link upperleg_M1_link
- removed link upperleg_M2_link
- removed link upperleg_M3_link
- added link entity_link, mass 0.1; visual box size=0.05 0.05 0.05
- added link world
- added link x_axis_link, mass 0.01; visual box size=0.1 0.05 0.05
- added link y_axis_link, mass 0.01; visual box size=0.05 0.1 0.05
Joints:
- removed joint basefoot_peg_M1_basefoot_peg_M1_joint_joint
- removed joint basefoot_peg_M2_basefoot_peg_M2_joint_joint
- removed joint basefoot_peg_M3_basefoot_peg_M3_joint_joint
- removed joint fixed
- removed joint head_upperlegM1_joint
- removed joint head_upperlegM2_joint
- removed joint head_upperlegM3_joint
- removed joint upperlegM1_lowerlegM1_joint
- removed joint upperlegM2_lowerlegM2_joint
- removed joint upperlegM3_lowerlegM3_joint
- added joint entity_link_joint: type fixed, parent y_axis_link, child entity_link, origin xyz=0 0 0.05 rpy=0 0 0
- added joint x_axis_joint: type prismatic, parent world, child x_axis_link, origin xyz=0 0 0 rpy=0.0 0.0 0.0, axis 1 0 0, limit lower=-5.0 upper=5.0 effort=10000 velocity=1
- added joint y_axis_joint: type prismatic, parent x_axis_link, child y_axis_link, origin xyz=0 0 0 rpy=0.0 0.0 0.0, axis 0 1 0, limit lower=-5.0 upper=5.0 effort=10000 velocity=1

Commit message: Added better performance plannar mover urdf

File: plannar_mover/urdf/plannar_mover.urdf (robot description, URDF)
Before this commit: robot gurdy, 4 links, 3 joints
Links:
- link x_axis_link: geometry collision box size=1.0 1.0 0.01; visual box size=1.0 1.0 0.01
- link y_axis_link: geometry collision box size=1.0 1.0 0.01; visual box size=1.0 1.0 0.01
Joints:
- joint entity_link_joint: origin xyz=0 0 0.05 rpy=0 0 0 -> xyz=0 0 0.025 rpy=0 0 0
- joint x_axis_joint: origin xyz=0 0 0 rpy=0.0 0.0 0.0 -> xyz=0 0 0.01 rpy=0.0 0.0 0.0
- joint y_axis_joint: origin xyz=0 0 0 rpy=0.0 0.0 0.0 -> xyz=0 0 0.01 rpy=0.0 0.0 0.0
